File: kicad/xiaozhi-with-ken-interface/xiaozhi-with-ken-interface.kicad_sch (KiCad schematic)
At the start: 9 parts, among them J1 Conn_01x04_Pin, U3 XDZ254-2-15-W-2.5-G1, U5 PM254-2-15-W-8.5, U6 adafruit-MAX98357

Commit message: add boot button to ESP32-S3 board, add speaker to xiaozhi, improve xiaozhi board schematic and routing.
Parts:
- added SPK1: FS-1540, FS-1540:BUZ-SMD_5P-L15.0-W15.0-P13.7-BL, symbol FS-1540:FS-1540
- added SW1, SW2: TSC015A03526A, TSC015A03526A:SW-SMD_4P-L4.5-W4.5-P3.00-LS6.8, symbol TSC015A03526A:TSC015A03526A
Connections:
- net +3V3: now also J1.2 (Pin_2), M1.VDD, U6.1 (Vin), U6.3 (~{SD_MODE})
- net BTN_C: now also SW2.2
- net BTN_D: now also SW1.2
- net GND: now also J1.1 (Pin_1), M1.GND, M1.L/R, U6.2 (GND), U6.4 (GAIN), SW1.3, SW1.4, SW2.3, SW2.4
- net I2C_B_SCL: now also J1.3 (Pin_3)
- net I2C_B_SDA: now also J1.4 (Pin_4)
- net I2S_A_SCK: now also M1.SCK
- net I2S_A_SD: now also M1.SD
- net I2S_A_WS: now also M1.WS
- net I2S_B_BCLK: now also U6.6 (BCLK)
- net I2S_B_DIN: now also U6.5 (DIN)
- net I2S_B_LRC: now also U6.7 (LRC)
- net at U6.8 (OUTP): now also SPK1.1 (+)
- net at U6.9 (OUTN): now also SPK1.2
- no-connect marks 4 -> 8
Other:
- note added: "BUTTONS"
- note added: "I2S MIC"
- note added: "I2S OUTPUT"
- note added: "OLED"
- note added: "SCL"
- note added: "SDA"
- note added: "SPEAKER"
- note added: "volume down"
- note added: "volume up"
- note removed: "Auto Flash"
- note removed: "ESP32-S3-WROOM-1"
- note removed: "POWER"
- note removed: "USB-UART"
- moved on the sheet: J1, M1, U6
