File: kicad/xiaozhi-with-ken-interface/xiaozhi-with-ken-interface.kicad_pcb (KiCad board)
At the start: 4 copper layers, 50.8 x 81.3 mm, 9 parts, among them J1 Conn_01x04_Pin, U3 XDZ254-2-15-W-2.5-G1, U5 PM254-2-15-W-8.5, U6 adafruit-MAX98357

Commit message: add boot button to ESP32-S3 board, add speaker to xiaozhi, improve xiaozhi board schematic and routing.
Parts:
- added SPK1: FS-1540, FS-1540:BUZ-SMD_5P-L15.0-W15.0-P13.7-BL, B.Cu at (83.8, 89.6)
- added SW1: TSC015A03526A, TSC015A03526A:SW-SMD_4P-L4.5-W4.5-P3.00-LS6.8, F.Cu at (102.9, 62.2)
- added SW2: TSC015A03526A, TSC015A03526A:SW-SMD_4P-L4.5-W4.5-P3.00-LS6.8, F.Cu at (64.8, 62.2)
- added kibuzzard-69756C5B: G***, kibuzzard-69756C5B, F.Cu at (69.8, 62.2)
- added kibuzzard-69756C68: G***, kibuzzard-69756C68, F.Cu at (97.8, 62.2)
Connections:
- J1 pad 1: unconnected-(J1-Pin_1-Pad1) -> GND
- J1 pad 2: unconnected-(J1-Pin_2-Pad2) -> +3V3
- J1 pad 3: unconnected-(J1-Pin_3-Pad3) -> /I2C_B_SCL
- J1 pad 4: unconnected-(J1-Pin_4-Pad4) -> /I2C_B_SDA
- M1 pad GND: unconnected-(M1-PadGND) -> GND
- M1 pad L/R: unconnected-(M1-PadL/R) -> GND
- M1 pad SCK: unconnected-(M1-PadSCK) -> /I2S_A_SCK
- M1 pad SD: unconnected-(M1-PadSD) -> /I2S_A_SD
- M1 pad VDD: unconnected-(M1-PadVDD) -> +3V3
- M1 pad WS: unconnected-(M1-PadWS) -> /I2S_A_WS
- U6 pad 1: unconnected-(U6-Vin-Pad1) -> +3V3
- U6 pad 2: unconnected-(U6-GND-Pad2) -> GND
- U6 pad 3: unconnected-(U6-~{SD_MODE}-Pad3) -> +3V3
- U6 pad 4: unconnected-(U6-GAIN-Pad4) -> GND
- U6 pad 5: unconnected-(U6-DIN-Pad5) -> /I2S_B_DIN
- U6 pad 6: unconnected-(U6-BCLK-Pad6) -> /I2S_B_BCLK
- U6 pad 7: unconnected-(U6-LRC-Pad7) -> /I2S_B_LRC
- U6 pad 8: unconnected-(U6-OUTP-Pad8) -> Net-(SPK1-+)
- U6 pad 9: unconnected-(U6-OUTN-Pad9) -> Net-(U6-OUTN)
Routing:
- net +3V3: track 91.0 -> 192.9 mm
- net /I2C_B_SDA: track 37.2 -> 92.9 mm
- net /I2C_B_SCL: track 38.3 -> 92.9 mm
- net /BTN_D: track 37.2 -> 80.9 mm
- net /BTN_C: track 38.6 -> 81.7 mm
- net Net-(U6-OUTN): track 0.00 -> 27.4 mm, vias 0 -> 2
- net /I2S_B_DIN: track 37.2 -> 62.7 mm
- net Net-(SPK1-+): track 0.00 -> 24.3 mm
- net /I2S_A_SD: track 37.2 -> 59.8 mm
- net /I2S_A_SCK: track 37.2 -> 59.8 mm
- net /I2S_A_WS: track 37.2 -> 59.8 mm
- net /I2S_B_BCLK: track 38.3 -> 56.0 mm
- net /I2S_B_LRC: track 37.2 -> 51.4 mm
Other:
- board text added: "version:1.0 date: 20260125"
- board text removed: "version:1.0 date: 20260124"

Commit message: small update
Parts:
- SPK1: moved to F.Cu
- moved SPK1 0.44 mm to (83.8, 89.2)
Routing:
- net +3V3: track 192.9 -> 175.1 mm, vias 0 -> 1
- net Net-(SPK1-+): track 24.3 -> 37.4 mm
- net Net-(U6-OUTN): track 27.4 -> 37.5 mm, vias 2 -> 0
- net /I2S_B_DIN: track 62.7 -> 61.6 mm
- net /I2C_A_SCL: track 32.2 -> 31.1 mm
- net /I2C_A_SDA: track 32.2 -> 31.1 mm
- net /I2S_B_BCLK: track 56.0 -> 55.0 mm
- net GND: vias 0 -> 32
Other:
- board text added: "BCLK"
- board text added: "DIN"
- board text added: "LRC"
- board text added: "SCK"
- board text added: "SD"
- board text added: "WS"
- board text removed: "I2S_A_SCK"
- board text removed: "I2S_A_SD"
- board text removed: "I2S_A_WS"
- board text removed: "I2S_B_BCLK"
- board text removed: "I2S_B_DIN"
- board text removed: "I2S_B_LRC"
