File: kicad/xiaozhi-with-ken-interface/xiaozhi-with-ken-interface.kicad_pcb (KiCad board)
At the start: 4 copper layers, 50.8 x 81.3 mm, 14 parts, among them J1 Conn_01x04_Pin, SW1 TSC015A03526A, SW2 TSC015A03526A, U3 XDZ254-2-15-W-2.5-G1, U5 PM254-2-15-W-8.5, U6 adafruit-MAX98357

Commit message: final adjust, send to pcb maker
Routing:
- net /I2S_B_DIN: track 61.6 -> 58.6 mm

Commit message: fix labels, update manufacture files
Other:
- board text added: "Xiaozhi AI with KEN Interface"
- board text removed: "Xiaozhi AI with KEN interface"
