File: kicad/template/template.kicad_pcb (KiCad board)
At the start: 4 copper layers, 50.8 x 81.3 mm, 6 parts, among them U3 XDZ254-2-15-W-2.5-G1, U5 PM254-2-15-W-8.5

Commit message: add text
Other:
- board text added: "Template for Extension board with EKN interface"
