File: kicad/display-with-ken-interface/display-with-ken-interface.kicad_sch (KiCad schematic)
At the start: 9 parts, among them J4 TFT_SPI, J5 Conn_01x08_Pin, U3 XDZ254-2-15-W-2.5-G1, U5 PM254-2-15-W-8.5

Commit message: display board is ready to send to pcb maker
Parts:
- added J1: Conn_01x07_Pin, Connector_PinHeader_2.54mm:PinHeader_1x07_P2.54mm_Vertical, symbol Connector:Conn_01x07_Pin
Connections:
- net +3V3: now also J1.1 (Pin_1), J1.6 (Pin_6)
- net GC9A01_DC: now also J1.2 (Pin_2)
- net GC9A01_RESET: now also J1.3 (Pin_3)
- net GC9A01_SCL: now also J1.5 (Pin_5)
- net GC9A01_SDA(MOSI): now also J1.4 (Pin_4)
- net GND: now also J1.7 (Pin_7)
Other:
- moved on the sheet: J4, JP1

Commit message: Update display-with-ken-interface.kicad_sch
Other:
- note added: "19"
- note added: "20"
Changed lines of the file:
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@@
+		)
+	)
+	(text "20"
+		(exclude_from_sim no)
+		(at 373.38 116.078 0)
+		(effects
+			(font
+				(size 1.27 1.27)
+			)
 		)
 	)
@@
 		)
 	)
+	(text "19"
+		(exclude_from_sim no)
+		(at 373.38 107.188 0)
+		(effects
+			(font
+				(size 1.27 1.27)
+			)
+		)
+	)
