File: kicad/esp32-s3-with-ken-interface/esp32-s3-with-ken-interface.kicad_sch (KiCad schematic)
At the start: 32 parts, among them J1 TYPE-C-31-M-12, Q1 UMH3N, SW1 TSC015A03526A, U1 CH340C, U2 AMS1117-3.3, U3 XDZ254-2-15-W-2.5-G1, U4 ESP32-S3-WROOM-1, U5 PM254-2-15-W-8.5

Commit message: add KiCad project for xiaozhi AI with KEN interface
Changed lines of the file:
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@@
 		)
 	)
-	(label "PWM_5"
+	(label "PWM_E"
 		(at 205.74 180.34 0)
 		(effects
@@
 		)
 	)
-	(label "PWM_4"
+	(label "PWM_D"
 		(at 85.09 171.45 0)
 		(effects
@@
 		)
 	)
-	(label "PWM_1"
+	(label "PWM_A"
 		(at 85.09 160.02 0)
 		(effects
@@
 		)
 	)
-	(label "PWM_6"
+	(label "PWM_F"
 		(at 85.09 179.07 0)
 		(effects
@@
 		)
 	)
-	(label "PWM_6"
+	(label "PWM_F"
 		(at 341.63 182.88 0)
 		(effects
@@
 		)
 	)
-	(label "PWM_5"
+	(label "PWM_E"
 		(at 341.63 180.34 0)
 		(effects
@@
 		)
 	)
-	(label "PWM_3"
+	(label "PWM_C"
 		(at 341.63 185.42 0)
 		(effects
@@
 		)
 	)
-	(label "PWM_1"
+	(label "PWM_A"
 		(at 309.88 182.88 0)
 		(effects
@@
 		)
 	)
-	(label "PWM_3"
+	(label "PWM_C"
 		(at 85.09 167.64 0)
 		(effects
@@
 		)
 	)
-	(label "PWM_2"
+	(label "PWM_B"
 		(at 238.76 185.42 0)
 		(effects
@@
 		)
 	)
-	(label "PWM_3"
+	(label "PWM_C"
 		(at 205.74 185.42 0)
 		(effects
@@
 		)
 	)
-	(label "PWM_4"
+	(label "PWM_D"
 		(at 341.63 187.96 0)
 		(effects
@@
 		)
 	)
-	(label "PWM_2"
+	(label "PWM_B"
 		(at 85.09 163.83 0)
 		(effects
@@
 		)
 	)
-	(label "PWM_5"
+	(label "PWM_E"
 		(at 85.09 175.26 0)
 		(effects
@@
 		)
 	)
-	(label "PWM_4"
+	(label "PWM_D"
 		(at 205.74 187.96 0)
 		(effects
@@
 		)
 	)
-	(label "PWM_2"
+	(label "PWM_B"
 		(at 309.88 185.42 0)
 		(effects
@@
 		)
 	)
-	(label "PWM_1"
+	(label "PWM_A"
 		(at 238.76 182.88 0)
 		(effects
@@
 		)
 	)
-	(label "PWM_6"
+	(label "PWM_F"
 		(at 205.74 182.88 0)
 		(effects

Commit message: add boot button to ESP32-S3 board, add speaker to xiaozhi, improve xiaozhi board schematic and routing.
Parts:
- added SW2: TSC015A03526A, TSC015A03526A:SW-SMD_4P-L4.5-W4.5-P3.00-LS6.8, symbol TSC015A03526A:TSC015A03526A
Connections:
- net GND: now also SW2.3, SW2.4
- net IO0: now also SW2.2
- no-connect marks 12 -> 13
Other:
- note added: "boot button"
Changed lines of the file:
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@@
 		)
 	)
+	(text "boot button"
+		(exclude_from_sim no)
+		(at 233.68 94.234 0)
+		(effects
+			(font
+				(size 1.27 1.27)
+			)
+		)
+	)
 	(text "options (or just use pwm pins)"
 		(exclude_from_sim no)
@@
 	)
 	(junction
+		(at 224.79 109.22)
+		(diameter 0)
+		(color 0 0 0 0)
+	)
+	(junction
 		(at 156.21 45.72)
 		(diameter 0)
@@
 	)
 	(no_connect
+		(at 228.6 101.6)
+	)
+	(no_connect
 		(at 77.47 34.29)
 	)
@@
 	(wire
 		(pts
-			(xy 334.01 35.56) (xy 327.66 35.56)
+			(xy 39.37 49.53) (xy 39.37 46.99)
 		)
 		(stroke
@@
 	(wire
 		(pts
-			(xy 39.37 49.53) (xy 39.37 46.99)
+			(xy 156.21 29.21) (xy 162.56 29.21)
 		)
 		(stroke
@@
 	(wire
 		(pts
-			(xy 156.21 29.21) (xy 162.56 29.21)
+			(xy 275.59 35.56) (xy 297.18 35.56)
 		)
 		(stroke
@@
 	(wire
 		(pts
-			(xy 275.59 35.56) (xy 297.18 35.56)
+			(xy 170.18 45.72) (xy 170.18 50.8)
 		)
 		(stroke
@@
 	(wire
 		(pts
-			(xy 170.18 45.72) (xy 170.18 50.8)
+			(xy 238.76 101.6) (xy 247.65 101.6)
 		)
 		(stroke
@@
 	(wire
 		(pts
-			(xy 334.01 38.1) (xy 327.66 38.1)
-		)
-		(stroke
-			(width 0)
-			(type default)
-		)
-	)
-	(wire
-		(pts
 			(xy 142.24 45.72) (xy 156.21 45.72)
 		)
@@
 	(wire
 		(pts
-			(xy 292.1 40.64) (xy 297.18 40.64)
-		)
-		(stroke
-			(width 0)
-			(type default)
-		)
-	)
-	(wire
-		(pts
 			(xy 217.17 157.48) (xy 198.12 157.48)
 		)
@@
 	(wire
 		(pts
-			(xy 242.57 92.71) (xy 260.35 92.71)
+			(xy 224.79 106.68) (xy 224.79 109.22)
 		)
 		(stroke
@@
 	(wire
 		(pts
+			(xy 327.66 35.56) (xy 344.17 35.56)
+		)
+		(stroke
+			(width 0)
+			(type default)
+		)
+	)
+	(wire
+		(pts
 			(xy 238.76 167.64) (xy 232.41 167.64)
 		)
@@
 	(wire
 		(pts
+			(xy 242.57 109.22) (xy 224.79 109.22)
+		)
+		(stroke
+			(width 0)
+			(type default)
+		)
+	)
+	(wire
+		(pts
 			(xy 205.74 228.6) (xy 222.25 228.6)
 		)
@@
 	(wire
 		(pts
-			(xy 242.57 95.25) (xy 260.35 95.25)
+			(xy 292.1 76.2) (xy 297.18 76.2)
 		)
 		(stroke
@@
 	(wire
 		(pts
-			(xy 292.1 76.2) (xy 297.18 76.2)
+			(xy 80.645 52.07) (xy 80.645 53.34)
 		)
 		(stroke
@@
 	(wire
 		(pts
-			(xy 80.645 52.07) (xy 80.645 53.34)
+			(xy 334.01 43.18) (xy 327.66 43.18)
 		)
 		(stroke
@@
 	(wire
 		(pts
-			(xy 334.01 43.18) (xy 327.66 43.18)
+			(xy 176.53 88.9) (xy 185.42 88.9)
 		)
 		(stroke
@@
 	(wire
 		(pts
-			(xy 176.53 88.9) (xy 185.42 88.9)
+			(xy 74.93 109.22) (xy 74.93 85.09)
 		)
 		(stroke
@@
 	(wire
 		(pts
-			(xy 74.93 109.22) (xy 74.93 85.09)
+			(xy 309.88 160.02) (xy 321.31 160.02)
 		)
 		(stroke
@@
 	(wire
 		(pts
-			(xy 309.88 160.02) (xy 321.31 160.02)
+			(xy 386.08 78.74) (xy 386.08 88.9)
 		)
 		(stroke
@@
 	(wire
 		(pts
-			(xy 386.08 78.74) (xy 386.08 88.9)
+			(xy 327.66 38.1) (xy 344.17 38.1)
 		)
 		(stroke
@@
 	(wire
 		(pts
+			(xy 238.76 106.68) (xy 242.57 106.68)
+		)
+		(stroke
+			(width 0)
+			(type default)
+		)
+	)
+	(wire
+		(pts
 			(xy 151.13 104.14) (xy 158.75 104.14)
 		)
@@
 	(wire
 		(pts
+			(xy 292.1 40.64) (xy 297.18 40.64)
+		)
+		(stroke
+			(width 0)
+			(type default)
+		)
+	)
+	(wire
+		(pts
 			(xy 39.37 29.21) (xy 39.37 26.67)
 		)
@@
 	(wire
 		(pts
+			(xy 228.6 106.68) (xy 224.79 106.68)
+		)
+		(stroke
+			(width 0)
+			(type default)
+		)
+	)
+	(wire
+		(pts
 			(xy 85.09 146.05) (xy 101.6 146.05)
 		)
@@
 	(wire
 		(pts
+			(xy 242.57 106.68) (xy 242.57 109.22)
+		)
+		(stroke
+			(width 0)
+			(type default)
+		)
+	)
+	(wire
+		(pts
 			(xy 38.1 39.37) (xy 41.91 39.37)
 		)
@@
 		)
 	)
+	(label "IO0"
+		(at 247.65 101.6 180)
+		(effects
+			(font
+				(size 1.27 1.27)
+			)
+			(justify right bottom)
+		)
+	)
 	(label "I2S_A_SD"
 		(at 27.94 198.12 0)
@@
 		)
 	)
-	(label "RXD0"
-		(at 260.35 95.25 180)
-		(effects
-			(font
-				(size 1.27 1.27)
-			)
-			(justify right bottom)
-		)
-	)
 	(label "IO1"
 		(at 292.1 43.18 180)
@@
 		)
 	)
-	(label "TXD0"
-		(at 260.35 92.71 180)
-		(effects
-			(font
-				(size 1.27 1.27)
-			)
-			(justify right bottom)
-		)
-	)
 	(label "IO40"
 		(at 334.01 66.04 0)
@@
 	)
 	(label "MCU_TX"
-		(at 242.57 92.71 0)
+		(at 344.17 35.56 0)
 		(effects
 			(font
@@
 	)
 	(label "MCU_RX"
-		(at 242.57 95.25 0)
+		(at 344.17 38.1 0)
 		(effects
 			(font
@@
 	)
 	(symbol
+		(lib_id "TSC015A03526A:TSC015A03526A")
+		(at 233.68 104.14 0)
+		(unit 1)
+		(exclude_from_sim no)
+		(in_bom yes)
+		(on_board yes)
+		(dnp no)
+		(fields_autoplaced yes)
+		(property "Reference" "SW2"
+			(at 233.68 96.52 0)
+			(effects
+				(font
+					(size 1.27 1.27)
+				)
+			)
+		)
+		(property "Value" "TSC015A03526A"
+			(at 233.68 99.06 0)
+			(effects
+				(font
+					(size 1.27 1.27)
+				)
+			)
+		)
+		(property "Footprint" "TSC015A03526A:SW-SMD_4P-L4.5-W4.5-P3.00-LS6.8"
+			(at 233.68 114.3 0)
+			(effects
+				(font
+					(size 1.27 1.27)
+				)
+				(hide yes)
+			)
+		)
+		(property "Datasheet" ""
+			(at 233.68 104.14 0)
+			(effects
+				(font
+					(size 1.27 1.27)
+				)
+				(hide yes)
+			)
+		)
+		(property "Description" ""
+			(at 233.68 104.14 0)
+			(effects
+				(font
+					(size 1.27 1.27)
+				)
+				(hide yes)
+			)
+		)
+		(property "LCSC Part" "C2888900"
+			(at 233.68 116.84 0)
+			(effects
+				(font
+					(size 1.27 1.27)
+				)
+				(hide yes)
+			)
+		)
+		(pin "1"
+		)
+		(pin "4"
+		)
+		(pin "3"
+		)
+		(pin "2"
+		)
+		(instances
+			(project "esp32-s3-with-ken-interface"
+				(path "/5edcefbe-9766-42c8-9529-28d0ec865573"
+					(reference "SW2")
+					(unit 1)
+				)
+			)
+		)
+	)
+	(symbol
 		(lib_id "power:+3.3V")
 		(at 100.33 71.12 0)
@@
 					(unit 1)
 				)
+			)
+		)
+	)
+	(symbol
+		(lib_id "power:GND")
+		(at 224.79 109.22 0)
+		(unit 1)
+		(exclude_from_sim no)
+		(in_bom yes)
+		(on_board yes)
+		(dnp no)
+		(property "Reference" "#PWR028"
+			(at 224.79 115.57 0)
+			(effects
+				(font
+					(size 1.27 1.27)
+				)
+				(hide yes)
+			)
+		)
+		(property "Value" "GND"
+			(at 224.79 113.03 0)
+			(effects
+				(font
+					(size 1.27 1.27)
+				)
+			)
+		)
+		(property "Footprint" ""
+			(at 224.79 109.22 0)
+			(effects
+				(font
+					(size 1.27 1.27)
+				)
+				(hide yes)
+			)
+		)
+		(property "Datasheet" ""
+			(at 224.79 109.22 0)
+			(effects
+				(font
+					(size 1.27 1.27)
+				)
+				(hide yes)
+			)
+		)
+		(property "Description" ""
+			(at 224.79 109.22 0)
+			(effects
+				(font
+					(size 1.27 1.27)
+				)
+				(hide yes)
+			)
+		)
+		(pin "1"
+		)
+		(instances
+			(project "esp32-s3-with-ken-interface"
+				(path "/5edcefbe-9766-42c8-9529-28d0ec865573"
+					(reference "#PWR028")
+					(unit 1)
+				)

Commit message: sda:14, scl:15 I2C oled display demo, and mic wave form demo
Other:
- note added: "Octal Flash / PSRAM variants (e.g. N16R8, N8R8) GPIO33-37 - Additionally occupied by Octal SPI lines. Do not use."
Changed lines of the file:
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@@
 	)
 	(rectangle
-		(start 15.24 257.81)
-		(end 242.57 281.94)
+		(start 15.24 246.38)
+		(end 297.18 281.94)
 		(stroke
 			(width 0)
@@
 	(rectangle
 		(start 130.81 205.74)
-		(end 242.57 254)
+		(end 242.57 243.84)
 		(stroke
 			(width 0)
@@
 	(rectangle
 		(start 15.24 128.27)
-		(end 128.27 254)
+		(end 128.27 243.84)
 		(stroke
 			(width 0)
@@
 	(text "GPIO0, GPIO3, GPIO45, GPIO46 : Strapping pins.\nGPIO26, GPIO27, GPIO28, GPIO29, GPIO30, GPIO31, GPIO32 : SPI0/1 interface connected to\nthe in-package flash and PSRAM, or recommended for the off-package flash and PSRAM."
 		(exclude_from_sim no)
-		(at 17.78 261.874 0)
+		(at 18.288 249.174 0)
 		(effects
 			(font
@@
 		)
 	)
+	(text "Octal Flash / PSRAM variants (e.g. N16R8, N8R8)\nGPIO33-37 - Additionally occupied by Octal SPI lines. Do not use."
+		(exclude_from_sim no)
+		(at 81.026 270.51 0)
+		(effects
+			(font
+				(size 2.54 2.54)
+			)
+		)
+	)
 	(text "bit clock"
 		(exclude_from_sim no)
@@
 	(text "options (or just use pwm pins)"
 		(exclude_from_sim no)
-		(at 156.464 225.298 0)
+		(at 152.654 212.598 0)
 		(effects
 			(font
@@
 	(text "for oled, etc. option"
 		(exclude_from_sim no)
-		(at 205.74 224.282 0)
+		(at 201.93 211.582 0)
 		(effects
 			(font
@@
 	(wire
 		(pts
-			(xy 156.21 240.03) (xy 172.72 240.03)
+			(xy 152.4 227.33) (xy 168.91 227.33)
 		)
 		(stroke
@@
 	(wire
 		(pts
-			(xy 156.21 236.22) (xy 172.72 236.22)
+			(xy 152.4 223.52) (xy 168.91 223.52)
 		)
 		(stroke
@@
 	(wire
 		(pts
-			(xy 205.74 228.6) (xy 222.25 228.6)
+			(xy 201.93 215.9) (xy 218.44 215.9)
 		)
 		(stroke
@@
 	(wire
 		(pts
-			(xy 205.74 232.41) (xy 222.25 232.41)
+			(xy 201.93 219.71) (xy 218.44 219.71)
 		)
 		(stroke
@@
 	(wire
 		(pts
-			(xy 156.21 228.6) (xy 172.72 228.6)
+			(xy 152.4 215.9) (xy 168.91 215.9)
 		)
 		(stroke
@@
 	(wire
 		(pts
-			(xy 156.21 232.41) (xy 172.72 232.41)
+			(xy 152.4 219.71) (xy 168.91 219.71)
 		)
 		(stroke
@@
 	)
 	(label "BTN_A"
-		(at 156.21 228.6 0)
+		(at 152.4 215.9 0)
 		(effects
 			(font
@@
 	)
 	(label "BTN_D"
-		(at 156.21 240.03 0)
+		(at 152.4 227.33 0)
 		(effects
 			(font
@@
 	)
 	(label "BTN_C"
-		(at 156.21 236.22 0)
+		(at 152.4 223.52 0)
 		(effects
 			(font
@@
 	)
 	(label "IO39"
-		(at 172.72 236.22 0)
+		(at 168.91 223.52 0)
 		(effects
 			(font
@@
 	)
 	(label "I2C_B_SCL"
-		(at 205.74 232.41 0)
+		(at 201.93 219.71 0)
 		(effects
 			(font
@@
 	)
 	(label "IO41"
-		(at 222.25 228.6 0)
+		(at 218.44 215.9 0)
 		(effects
 			(font
@@
 	)
 	(label "BTN_B"
-		(at 156.21 232.41 0)
+		(at 152.4 219.71 0)
 		(effects
 			(font
@@
 	)
 	(label "IO14"
-		(at 172.72 228.6 0)
+		(at 168.91 215.9 0)
 		(effects
 			(font
@@
 	)
 	(label "IO21"
-		(at 172.72 232.41 0)
+		(at 168.91 219.71 0)
 		(effects
 			(font
@@
 	)
 	(label "IO42"
-		(at 222.25 232.41 0)
+		(at 218.44 219.71 0)
 		(effects
 			(font
@@
 	)
 	(label "IO40"
-		(at 172.72 240.03 0)
+		(at 168.91 227.33 0)
 		(effects
 			(font
@@
 	)
 	(label "I2C_B_SDA"
-		(at 205.74 228.6 0)
+		(at 201.93 215.9 0)
 		(effects
 			(font

Commit message: add reset button
Parts:
- removed H3, H4: MountHole, MountingHole:MountingHole_3.2mm_M3_DIN965_Pad, symbol Mechanical:MountingHole_Pad
- added SW3: TSC015A03526A, TSC015A03526A:SW-SMD_4P-L4.5-W4.5-P3.00-LS6.8, symbol TSC015A03526A:TSC015A03526A
Connections:
- net EN: now also SW3.2
- net GND: now also SW3.3, SW3.4
- no-connect marks 13 -> 12
Other:
- note added: "reset"
- moved on the sheet: SW2
